File: digital lockin.brd (EAGLE design)
At the start: 76.2 x 94.9 mm, 24 parts, among them IC1 OPA2650E, IC2 LM358D, T2 NPN, U2 RASPBERRY_PICOSMD-TH, U5 TL431AIDBZR

Commit message: Add files via upload
Parts:
- moved C1 20.8 mm to (48.0, 25.9), turned to 0 degrees
- moved R9 20.0 mm to (42.4, 14.2), turned to 180 degrees
- moved C3 11.8 mm to (62.2, 17.8)
- moved R5 11.5 mm to (63.2, 29.7)
- moved R7 10.4 mm to (71.4, 14.7)
- moved PD1 7.22 mm to (39.9, 19.1), turned to 0 degrees
- moved C10 6.83 mm to (47.8, 10.2), turned to 270 degrees
- moved IC1 6.47 mm to (54.4, 17.5)
- moved R3 6.37 mm to (47.0, 18.8), turned to 180 degrees
- moved R6 0.72 mm to (58.2, 22.4), turned to 180 degrees
Connections:
- removed net V+: IC1.8
- removed net V-: IC1.4
- new net N$1: C3.1, IC1.7, R6.1
- new net N$11: C10.1, IC1.4, PD1.A
- new net N$13: C8.1, IC1.8
- new net N$2: C3.2, IC1.6, R7.1
- new net N$4: C2.2, R7.2
- new net N$5: C2.1, IC1.5, R5.2
- new net N$6: C1.2, IC1.1, R3.1, R5.1
- new net N$7: C1.1, IC1.2, PD1.K, R3.2, R6.2
- new net N$8: C10.2, IC1.3, R9.1
- net GND: now also C8.2
Routing:
- net N$7: track 0.00 -> 17.7 mm
- net N$11: track 0.00 -> 5.33 mm
- net N$6: track 0.00 -> 4.60 mm
- net N$2: track 0.00 -> 0.53 mm

Commit message: Add files via upload
Parts:
- moved R5 18.2 mm to (54.1, 14.0), turned to 0 degrees
- moved C2 10.3 mm to (61.2, 16.0), turned to 0 degrees
- moved R3 6.91 mm to (51.1, 24.4), turned to 270 degrees
- moved C1 6.78 mm to (54.6, 24.4), turned to 90 degrees
- moved R7 6.14 mm to (65.8, 17.3)
- moved PD1 4.60 mm to (44.5, 19.6), turned to 90 degrees
- moved C10 2.87 mm to (45.7, 12.2), turned to 180 degrees
- moved R9 1.83 mm to (40.9, 15.2)
- moved C3 1.83 mm to (61.2, 19.3), turned to 0 degrees
- moved R6 1.44 mm to (59.2, 23.4)
Routing:
- net N$6: track 4.60 -> 31.9 mm, vias 0 -> 2
- net N$8: track 0.00 -> 18.2 mm
- net N$1: track 0.00 -> 11.3 mm
- net N$2: track 0.53 -> 11.5 mm
- net N$7: track 17.7 -> 28.4 mm
- net N$5: track 0.00 -> 9.79 mm
- net N$11: track 5.33 -> 0.00 mm
- net N$4: track 0.00 -> 3.94 mm

Commit message: Add files via upload
Parts:
- moved C8 14.7 mm to (59.4, 19.3), turned to 0 degrees
- moved C3 4.06 mm to (65.3, 19.3)
- moved R6 3.09 mm to (62.2, 22.9)
- moved C2 3.05 mm to (64.3, 16.0)
- moved R7 2.03 mm to (67.8, 17.3)
- moved C10 1.61 mm to (44.2, 11.7)
Routing:
- net N$11: track 0.00 -> 28.5 mm
- net N$7: track 28.4 -> 31.5 mm
- net N$5: track 9.79 -> 12.8 mm
- net N$13: track 0.00 -> 2.82 mm
- net N$8: track 18.2 -> 16.1 mm
- net N$2: track 11.5 -> 13.6 mm
- net N$1: track 11.3 -> 12.9 mm
- net N$6: track 31.9 -> 30.6 mm, vias 2 -> 3
- net N$4: track 3.94 -> 2.93 mm
